File: cynaroides.kicad_pcb (KiCad board)
At the start: 4 copper layers, 145.3 x 115.1 mm, 136 parts, among them J1 USB_C_Receptacle_USB2.0, J2 MJ-4PP-9, Q1 DTC123J, SW1 SW_Push, SW10 SW_Push, SW11 SW_Push, SW12 SW_Push, SW13 SW_Push, SW14 SW_Push, SW15 SW_Push, SW16 SW_Push, SW17 SW_Push, SW18 SW_Push, SW19 SW_Push, SW2 SW_Push, SW20 SW_Push, SW21 SW_Push, SW22 SW_Push, SW23 SW_Push, SW24 SW_Push, SW25 SW_Push, SW26 SW_Push, SW27 SW_Push, SW28 SW_Push, SW29 SW_Push, SW3 SW_Push, SW30 SW_Push, SW31 SW_Push, SW4 SW_Push, SW5 SW_Push, SW6 SW_Push, SW7 SW_Push, SW8 SW_Push, SW9 SW_Push, U1 USBLC6-2SC6, U2 STM32F411RCTx, U3 25LCxxx, U4 MCP1700-3302E_SOT23, Y1 Crystal_GND24_Small

Commit message: Adding pcb files
Parts:
- moved D3 31.0 mm to (73.0, 82.9), turned to 180 degrees
- moved SW13 29.1 mm to (203.5, 70.2)
- moved SW31 29.1 mm to (175.7, 125.8)
- moved SW7 29.1 mm to (203.5, 51.2)
- moved D27 29.1 mm to (192.5, 106.4)
- moved D9 29.1 mm to (192.5, 47.5)
- moved SW19 29.1 mm to (203.5, 89.3)
- moved SW25 29.1 mm to (203.5, 108.3)
- moved D10 29.1 mm to (113.9, 65.3)
- moved D34 29.1 mm to (105.9, 59.9)
- moved D36 29.1 mm to (144.0, 55.1)
- moved D43 29.1 mm to (144.0, 74.2)
- moved D45 29.1 mm to (105.9, 78.9)
- moved D46 29.1 mm to (105.9, 98.0)
- moved SW28 29.1 mm to (109.9, 126.6)
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Routing:
- net Net-(D3-Pad1): track 4.80 -> 8.23 mm
- net Net-(D3-Pad2): track 9.82 -> 12.3 mm
- net ROW0: track 115.7 -> 117.4 mm
- net SCL: track 33.5 -> 32.5 mm
